File: Devboard/devboard.brd (EAGLE design)
At the start: 100 x 70 mm, 89 parts, among them J1 USB-MICROB-2, J10 MJ-2509N, J11 MJ-2509N, J12 MJ-2509N, J13 MJ-2509N, J14 1x8M, J15 1x8F, J16 1x8F, J17 1x2M, J2 1x2M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

Commit message: Increased motor driver current
Parts:
- R6, R7, R8, R9: value 0.43R -> 0.39R
Changed lines of the file:
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@@
 <attribute name="PROD_ID" value="TRANS-11308" x="6.35" y="21.59" size="1.778" layer="27" display="off"/>
 </element>
-<element name="R6" library="vibhud" library_urn="urn:adsk.eagle:library:2530795" package="0805" package3d_urn="urn:adsk.eagle:package:2531030/1" value="0.43R" x="72.39" y="20.32" smashed="yes" rot="R90">
-<attribute name="NAME" x="72.136" y="17.145" size="0.6096" layer="25" font="vector" ratio="20" rot="R90" align="bottom-center"/>
+<element name="R6" library="vibhud" library_urn="urn:adsk.eagle:library:2530795" package="0805" package3d_urn="urn:adsk.eagle:package:2531030/1" value="0.39R" x="72.39" y="20.32" smashed="yes" rot="R90">
+<attribute name="NAME" x="72.39" y="21.971" size="0.6096" layer="25" font="vector" ratio="20" align="bottom-center"/>
 <attribute name="PROD_ID" value=" " x="72.39" y="20.32" size="1.778" layer="27" rot="R90" display="off"/>
-<attribute name="VALUE" x="72.644" y="17.145" size="0.6096" layer="27" font="vector" ratio="20" rot="R90" align="top-center"/>
+<attribute name="VALUE" x="72.644" y="18.669" size="0.6096" layer="27" font="vector" ratio="20" align="top-center"/>
 </element>
-<element name="R9" library="vibhud" library_urn="urn:adsk.eagle:library:2530795" package="0805" package3d_urn="urn:adsk.eagle:package:2531030/1" value="0.43R" x="61.595" y="20.32" smashed="yes" rot="R90">
-<attribute name="NAME" x="62.357" y="17.78" size="0.6096" layer="25" font="vector" ratio="20" rot="R90" align="bottom-center"/>
+<element name="R9" library="vibhud" library_urn="urn:adsk.eagle:library:2530795" package="0805" package3d_urn="urn:adsk.eagle:package:2531030/1" value="0.39R" x="61.595" y="20.32" smashed="yes" rot="R90">
+<attribute name="NAME" x="61.595" y="21.971" size="0.6096" layer="25" font="vector" ratio="20" align="bottom-center"/>
 <attribute name="PROD_ID" value=" " x="61.595" y="20.32" size="1.778" layer="27" rot="R90" display="off"/>
-<attribute name="VALUE" x="62.611" y="17.78" size="0.6096" layer="27" font="vector" ratio="20" rot="R90" align="top-center"/>
+<attribute name="VALUE" x="61.595" y="18.542" size="0.6096" layer="27" font="vector" ratio="20" align="top-center"/>
 </element>
 <element name="R2" library="vibhud" library_urn="urn:adsk.eagle:library:2530795" package="0805" package3d_urn="urn:adsk.eagle:package:2531030/1" value="220R" x="82.55" y="59.69" smashed="yes">
@@
 <attribute name="VALUE" x="84.328" y="59.69" size="0.6096" layer="27" font="vector" ratio="20" rot="R90" align="top-center"/>
 </element>
-<element name="R8" library="vibhud" library_urn="urn:adsk.eagle:library:2530795" package="0805" package3d_urn="urn:adsk.eagle:package:2531030/1" value="0.43R" x="59.055" y="20.32" smashed="yes" rot="R90">
-<attribute name="NAME" x="58.166" y="17.78" size="0.6096" layer="25" font="vector" ratio="20" rot="R90" align="bottom-center"/>
+<element name="R8" library="vibhud" library_urn="urn:adsk.eagle:library:2530795" package="0805" package3d_urn="urn:adsk.eagle:package:2531030/1" value="0.39R" x="59.055" y="20.32" smashed="yes" rot="R90">
+<attribute name="NAME" x="59.055" y="21.971" size="0.6096" layer="25" font="vector" ratio="20" align="bottom-center"/>
 <attribute name="PROD_ID" value=" " x="59.055" y="20.32" size="1.778" layer="27" rot="R90" display="off"/>
-<attribute name="VALUE" x="58.674" y="17.399" size="0.6096" layer="27" font="vector" ratio="20" rot="R90" align="top-center"/>
+<attribute name="VALUE" x="59.055" y="18.542" size="0.6096" layer="27" font="vector" ratio="20" align="top-center"/>
 </element>
 <element name="R5" library="vibhud" library_urn="urn:adsk.eagle:library:2530795" package="0805" package3d_urn="urn:adsk.eagle:package:2531030/1" value="10k" x="8.89" y="27.305" smashed="yes" rot="R270">
@@
 <attribute name="VALUE" x="84.328" y="66.04" size="0.6096" layer="27" font="vector" ratio="20" rot="R90" align="top-center"/>
 </element>
-<element name="R7" library="vibhud" library_urn="urn:adsk.eagle:library:2530795" package="0805" package3d_urn="urn:adsk.eagle:package:2531030/1" value="0.43R" x="76.2" y="20.32" smashed="yes" rot="R90">
-<attribute name="NAME" x="75.946" y="17.145" size="0.6096" layer="25" font="vector" ratio="20" rot="R90" align="bottom-center"/>
+<element name="R7" library="vibhud" library_urn="urn:adsk.eagle:library:2530795" package="0805" package3d_urn="urn:adsk.eagle:package:2531030/1" value="0.39R" x="76.2" y="20.32" smashed="yes" rot="R90">
+<attribute name="NAME" x="76.2" y="21.971" size="0.6096" layer="25" font="vector" ratio="20" align="bottom-center"/>
 <attribute name="PROD_ID" value=" " x="76.2" y="20.32" size="1.778" layer="27" rot="R90" display="off"/>
-<attribute name="VALUE" x="76.454" y="17.145" size="0.6096" layer="27" font="vector" ratio="20" rot="R90" align="top-center"/>
+<attribute name="VALUE" x="77.216" y="20.32" size="0.6096" layer="27" font="vector" ratio="20" rot="R90" align="top-center"/>
 </element>
 <element name="R4" library="vibhud" library_urn="urn:adsk.eagle:library:2530795" package="0805" package3d_urn="urn:adsk.eagle:package:2531030/1" value="10k" x="10.16" y="43.18" smashed="yes" rot="R90">

Commit message: Final changes to dev board for manufacture
Parts:
- FLASH, RESET: value MOMENTARY-SWITCH-SPST-PTH-6.0MM -> MOMENTARY-SWITCH-SPST-SMD-6.0X3.5MM; device vibhud:TACTILE_SWITCH_PTH_6.0MM -> vibhud:TACTILE_SWITCH_SMD_6.0X3.5MM
- moved FLASH 19.1 mm to (31.8, 61.6), turned to 180 degrees
- moved D4 6.10 mm to (30.9, 45.2), turned to 270 degrees
- moved RESET 2.69 mm to (31.8, 66.0)
Connections:
- net GND: now also FLASH.2, RESET.2; no longer FLASH.3, RESET.3
Routing:
- net PWR_LED: track 5.61 -> 12.8 mm
- net GPIO0: track 61.4 -> 56.3 mm, vias 1 -> 3
- net PWM7: track 54.0 -> 58.6 mm
- net 3.3V: track 158.2 -> 162.6 mm
- net RESET: track 21.5 -> 25.6 mm
- net PWM6: track 52.0 -> 54.3 mm
- net PWM5: track 54.6 -> 55.8 mm
- net PWM4: track 55.8 -> 55.2 mm
- net GND: vias 22 -> 23
Other:
- board text added: "Motors"
- board text added: "PWM"

Commit message: Changed fuse rating
Parts:
- F1: value 8V/2.2A -> 6V/2A
Changed lines of the file:
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@@
 <attribute name="NAME" x="91.313" y="45.339" size="0.6096" layer="25" font="vector" ratio="18" rot="R180"/>
 </element>
-<element name="F1" library="vibhud" library_urn="urn:adsk.eagle:library:2530795" package="1206" package3d_urn="urn:adsk.eagle:package:2531016/1" value="8V/2.2A" x="12.7" y="27.305" smashed="yes" rot="R90">
+<element name="F1" library="vibhud" library_urn="urn:adsk.eagle:library:2530795" package="1206" package3d_urn="urn:adsk.eagle:package:2531016/1" value="6V/2A" x="12.7" y="27.305" smashed="yes" rot="R90">
 <attribute name="NAME" x="11.303" y="27.305" size="0.6096" layer="25" font="vector" ratio="20" rot="R90" align="bottom-center"/>
 <attribute name="PROD_ID" value="RES-08585" x="12.7" y="27.305" size="1.778" layer="27" rot="R90" display="off"/>
