File: Devboard_1.1/devboard.brd (EAGLE design)
At the start: 100 x 70 mm, 89 parts, among them J1 USB-MICROB-2, J10 MJ-2509N, J11 MJ-2509N, J12 MJ-2509N, J13 MJ-2509N, J14 1x8M, J15 1x8F, J16 1x8F, J17 1x2M, J2 1x2M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

Commit message: Updates to 1.1 board
Parts:
- added C12: 10uF, vibhud:C1206
- added D3: Blue, vibhud:CHIPLED_0805_NOOUTLINE
- added R10: 51R, vibhud:0805
- added R11: 1k, vibhud:0805
- added U5: PCA9634D, vibhud:SOP65P640X110-20
- RN1, RN2, RN3, RN4, RN5, RN6, RN7, RN8, RN9: device vibhud:EXBS8V -> vibhud:EXB38V
- moved R2 19.6 mm to (63.5, 64.1), turned to 270 degrees
- moved S1 17.8 mm to (84.5, 64.1)
- moved R3 15.9 mm to (66.7, 64.1), turned to 270 degrees
- moved R1 12.8 mm to (69.8, 64.1), turned to 270 degrees
- moved RN2 6.02 mm to (85.1, 40.0), turned to 270 degrees
- moved RN1 4.98 mm to (84.5, 57.9), turned to 270 degrees
- moved C5 3.58 mm to (72.4, 58.2), turned to 180 degrees
- moved RN9 1.42 mm to (68.5, 58.7)
Connections:
- new net N$12: D1.4, R10.1
- new net N$13: D3.A, R11.2
- new net N$14: J13.2, J9.VBUS
- new net N$32: J10.2, J6.VBUS
- new net N$33: J11.2, J7.VBUS
- new net N$34: J12.2, J8.VBUS
- net 3.3V: now also C12.1, R10.2, U5.20; no longer D1.4
- net GND: now also C12.2, D3.C, U5.1, U5.10, U5.15, U5.16, U5.17, U5.2, U5.3, U5.4, U5.5
- net GPIO15: now also R11.1
- net MOT_0P: no longer J6.VBUS
- net MOT_1N: now also U2.P$5; no longer U2.P$7
- net MOT_1P: now also U2.P$7; no longer J7.VBUS, U2.P$5
- net MOT_2P: no longer J8.VBUS
- net MOT_3N: now also U3.P$5; no longer U3.P$7
- net MOT_3P: now also U3.P$7; no longer J9.VBUS, U3.P$5
- net PWM0: now also U5.6
- net PWM1: now also U5.7
- net PWM2: now also U5.8
- net PWM3: now also U5.9
- net PWM4: now also U5.11
- net PWM5: now also U5.12
- net PWM6: now also U5.13
- net PWM7: now also U5.14
- net SCL: now also U5.18
- net SDA: now also U5.19
Routing:
- net 3.3V: track 162.6 -> 130.7 mm
- net GPIO0: track 56.3 -> 26.1 mm, vias 3 -> 1
- net MOT_1N: track 110.5 -> 82.1 mm, vias 2 -> 1
- net MOT_3N: track 77.2 -> 50.8 mm, vias 1 -> 0
- net GPIO2: track 65.2 -> 39.2 mm, vias 2 -> 1
- net GPIO13: track 60.0 -> 35.1 mm, vias 2 -> 1
- net GPIO12: track 58.2 -> 33.4 mm, vias 2 -> 1
- net MOT_0N: track 125.6 -> 104.0 mm
- net MOT_2N: track 96.1 -> 76.7 mm
- net RESET: track 25.6 -> 6.30 mm
- net MOT_3P: track 68.8 -> 49.9 mm, vias 2 -> 1
- net USB_DTR: track 15.3 -> 0.00 mm
- net N$8: track 13.5 -> 0.00 mm
- net MOT_1P: track 95.8 -> 82.7 mm, vias 2 -> 1
- net PWR_LED: track 12.8 -> 0.00 mm
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