File: Devboard_1.1/devboard.brd (EAGLE design)
At the start: 100 x 70 mm, 94 parts, among them J1 USB-MICROB-2, J10 MJ-2509N, J11 MJ-2509N, J12 MJ-2509N, J13 MJ-2509N, J14 1x8M, J15 1x8F, J16 1x8F, J17 1x2M, J2 1x2M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

Commit message: Updated 1.1 board
Parts:
- removed C12: 10uF, vibhud:C1206
- removed J17: 1x2M, vibhud:1X02_LOCK_LONGPADS
- removed U5: PCA9634D, vibhud:SOP65P640X110-20
- added J19: 1x8M, vibhud:1X06_LOCK
- C1, C10, C11, C2, C3, C4, C5, C6, C7, C8, C9: device vibhud:C1206 -> vibhud:C0805
- RN1, RN2, RN3, RN4, RN5, RN7, RN8, RN9: device vibhud:EXB38V -> vibhud:EXB28V
- RN6: device vibhud:EXB38V -> vibhud:EXBN8V
- moved LOGO1 63.6 mm to (33.0, 65.4)
- moved FLASH 38.9 mm to (7.62, 31.1)
- moved RESET 38.4 mm to (7.62, 36.2)
- moved D4 17.9 mm to (15.5, 54.5), turned to 90 degrees
- moved R4 16.3 mm to (26.3, 45.7), turned to 0 degrees
- moved U4 8.98 mm to (27.3, 41.9)
- moved C2 8.92 mm to (31.8, 41.9)
- moved R5 8.89 mm to (8.89, 18.4)
- moved C1 8.81 mm to (22.4, 41.8)
- moved J2 7.62 mm to (5.84, 22.9), turned to 0 degrees
- moved F1 6.35 mm to (12.7, 21.0)
- moved D2 6.35 mm to (12.7, 12.1)
- moved Q1 6.35 mm to (6.35, 15.2)
- moved R10 6.02 mm to (69.2, 62.9), turned to 180 degrees
- moved R1 5.68 mm to (64.8, 66.7), turned to 180 degrees
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Connections:
- removed net N$31: J16.1, J17.2
- net 3.3V: no longer C12.1, U5.20
- net CH_PD: now also RN8.6; no longer RN8.7
- net GND: now also J19.1; no longer C12.2, U5.1, U5.10, U5.15, U5.16, U5.17, U5.2, U5.3, U5.4, U5.5
- net GPIO0: now also RN8.8; no longer RN8.5
- net GPIO14: now also RN8.5; no longer RN8.6
- net PWM0: no longer U5.6
- net PWM1: no longer U5.7
- net PWM2: no longer U5.8
- net PWM3: no longer U5.9
- net PWM4: no longer U5.11
- net PWM5: no longer U5.12
- net PWM6: no longer U5.13
- net PWM7: no longer U5.14
- net RESET: now also RN8.7; no longer RN8.8
- net SCL: no longer U5.18
- net SDA: no longer U5.19
- net TXD0: now also J19.5
- net USB_RXD: now also J19.4
- net V_USB: now also J16.1, J19.3; no longer J17.1
Routing:
- net GPIO0: track 26.1 -> 87.8 mm, vias 1 -> 3
- net N$32: track 0.00 -> 54.9 mm, vias 0 -> 1
- net N$33: track 0.00 -> 53.5 mm, vias 0 -> 1
- net RESET: track 6.30 -> 59.0 mm, vias 0 -> 2
- net N$34: track 0.00 -> 49.6 mm, vias 0 -> 1
- net N$14: track 0.00 -> 45.7 mm, vias 0 -> 1
- net GND: track 114.0 -> 158.8 mm
- net DTR: track 0.00 -> 37.0 mm
- net GPIO14: track 30.1 -> 65.5 mm
- net MOT_3N: track 50.8 -> 79.4 mm, vias 0 -> 1
- net USB_RXD: track 0.00 -> 27.9 mm
- net TXD0: track 39.9 -> 67.6 mm
- net MOT_1N: track 82.1 -> 108.7 mm, vias 1 -> 2
- net 3.3V: track 130.7 -> 155.9 mm, vias 1 -> 3
- net MOT_3P: track 49.9 -> 71.9 mm, vias 1 -> 3
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Other:
- board text added: "Kadah - June 2018"
- board text added: "VihHub Dev Board v1.1"
- board text removed: "May 2018"
- board text removed: "VihHub Dev Board v1.0"

Commit message: Updates to 1.1 board
Parts:
- added U$1: DICKBUTT, vibhud:DICKBUTT
- F1: value 6V/2A -> 16V/2.2A; device vibhud:1206 -> vibhud:FUSC7035X90
- RN6: device vibhud:EXBN8V -> vibhud:EXB28V
- moved C13 7.10 mm to (24.8, 34.3), turned to 90 degrees
- moved R4 6.66 mm to (29.7, 40.0), turned to 180 degrees
- moved R5 2.97 mm to (9.91, 15.6), turned to 180 degrees
- moved C2 2.29 mm to (33.0, 43.8)
- moved C1 2.29 mm to (23.6, 43.7)
- moved U4 2.29 mm to (28.6, 43.8)
- moved Q1 1.80 mm to (5.08, 16.5), turned to 90 degrees
- moved D2 1.65 mm to (11.0, 12.1), turned to 0 degrees
- moved F1 1.28 mm to (12.6, 22.2)
- moved J2 0.76 mm to (5.84, 22.1), turned to 90 degrees
- moved D3 0.76 mm to (67.2, 27.3)
- moved R11 0.76 mm to (67.2, 22.9)
- renumbered J19 to FTDI
Connections:
- net 3.3V: now also U1.16, U1.17
- net GND: no longer U1.16, U1.17
Routing:
- net GND: track 158.8 -> 142.2 mm, vias 23 -> 25
- net 3.3V: track 155.9 -> 164.1 mm
- net GPIO0: track 87.8 -> 80.5 mm
- net V_USB: track 69.1 -> 64.2 mm
- net N$5: track 10.8 -> 14.9 mm
- net 5V: track 104.7 -> 101.1 mm
- net N$14: track 45.7 -> 48.5 mm
- net N$35: track 12.7 -> 10.6 mm
- net N$1: track 5.92 -> 4.01 mm
- net MOT_1P: track 92.9 -> 91.8 mm
- net MOT_2P: track 82.1 -> 81.0 mm
- net MOT_0P: track 107.6 -> 106.5 mm
- net MOT_3P: track 71.9 -> 70.9 mm
- net GPIO15: track 80.5 -> 81.3 mm
- net DTR: track 37.0 -> 37.6 mm
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Other:
- board text added: "+"
- board text added: "-"
- board text added: "B+"
- board text added: "B-"
- board text added: "Black"
- board text added: "Green"
- board text added: "RXD"
- board text added: "TXD"
- board text added: "VCC"
- board text removed: "BAT+"

Commit message: 1.1 board finalizations
Parts:
- added U$2: JASX_LOGO_LARGE, vibhud:JASX_LOGO
- U$1: value DICKBUTT -> DICKBUTTCOPPER; device vibhud:DICKBUTT -> vibhud:DICKBUTT_COPPER
- moved U$1 69.0 mm to (14.6, 31.1), flipped to the bottom
Changed lines of the file:
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@@
 </element>
 <element name="C3" library="vibhud" library_urn="urn:adsk.eagle:library:2530795" package="C0805" package3d_urn="urn:adsk.eagle:package:2531036/1" value="10uF" x="46.355" y="40.64" smashed="yes">
-<attribute name="NAME" x="46.355" y="38.4175" size="0.8128" layer="25" font="vector" ratio="10" align="center"/>
-<attribute name="VALUE" x="46.736" y="37.2745" size="0.8128" layer="27" font="vector" ratio="10" align="center"/>
+<attribute name="NAME" x="48.26" y="40.9575" size="0.8128" layer="25" font="vector" ratio="10" align="center"/>
+<attribute name="VALUE" x="48.895" y="39.8145" size="0.8128" layer="27" font="vector" ratio="10" align="center"/>
 </element>
 <element name="C4" library="vibhud" library_urn="urn:adsk.eagle:library:2530795" package="C0805" package3d_urn="urn:adsk.eagle:package:2531036/1" value="1.0uF" x="43.815" y="40.64" smashed="yes">
-<attribute name="NAME" x="43.815" y="38.4175" size="0.8128" layer="25" font="vector" ratio="10" align="center"/>
-<attribute name="VALUE" x="43.434" y="37.2745" size="0.8128" layer="27" font="vector" ratio="10" align="center"/>
+<attribute name="NAME" x="41.91" y="40.9575" size="0.8128" layer="25" font="vector" ratio="10" align="center"/>
+<attribute name="VALUE" x="41.275" y="39.8145" size="0.8128" layer="27" font="vector" ratio="10" align="center"/>
 </element>
 <element name="C5" library="vibhud" library_urn="urn:adsk.eagle:library:2530795" package="C0805" package3d_urn="urn:adsk.eagle:package:2531036/1" value="10uF" x="73.406" y="57.277" rot="R90"/>
@@
 <attribute name="NAME" x="12.065" y="41.783" size="1.016" layer="25" font="vector" ratio="20" align="top-center"/>
 </element>
-<element name="U$1" library="vibhud" library_urn="urn:adsk.eagle:library:2530795" package="DICKBUTT" value="DICKBUTT" x="82.55" y="19.05"/>
+<element name="U$2" library="vibhud" library_urn="urn:adsk.eagle:library:2530795" package="JASX_LOGO" value="JASX_LOGO_LARGE" x="41.021" y="32.512"/>
+<element name="U$1" library="vibhud" library_urn="urn:adsk.eagle:library:2530795" package="DICKBUTT_COPPER" value="DICKBUTTCOPPER" x="14.605" y="31.115" rot="MR0"/>
 </elements>
 <signals>
@@
 <wire x1="12.73" y1="4.786" x2="12.73" y2="3.586" width="0.4064" layer="1"/>
 <via x="45.085" y="38.481" extent="1-16" drill="0.35"/>
-<via x="42.545" y="28.575" extent="1-16" drill="0.35"/>
+<via x="42.672" y="27.686" extent="1-16" drill="0.35"/>
 <contactref element="FLASH" pad="2"/>
 <contactref element="J4" pad="8"/>

Commit message: 1.1 dev board RTM
Routing:
- net 5V: track 101.1 -> 133.5 mm
- net V_USB: track 64.2 -> 69.3 mm
Changed lines of the file:
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@@
 <wire x1="0" y1="70" x2="0" y2="0" width="0" layer="20"/>
 <text x="7.239" y="65.913" size="1.27" layer="21" font="vector" ratio="20">VihHub Dev Board v1.1</text>
-<dimension x1="0" y1="0" x2="0" y2="70" x3="-5" y3="35" textsize="1.778" layer="1"/>
-<dimension x1="0" y1="70" x2="100" y2="70" x3="50" y3="75" textsize="1.778" layer="1"/>
+<dimension x1="0" y1="0" x2="0" y2="70" x3="-5" y3="35" textsize="1.778" layer="51"/>
+<dimension x1="0" y1="70" x2="100" y2="70" x3="50" y3="75" textsize="1.778" layer="51"/>
 <text x="7.62" y="64.77" size="0.8128" layer="21" font="vector" ratio="20">Kadah - June 2018</text>
 <hole x="97" y="3" drill="3.175"/>
@@
 <wire x1="65.67" y1="66.675" x2="66.675" y2="66.675" width="0.254" layer="1"/>
 <wire x1="66.675" y1="66.675" x2="67.945" y2="67.945" width="0.254" layer="1"/>
-<wire x1="74.815" y1="67.945" x2="77.9" y2="64.86" width="0.254" layer="1"/>
-<wire x1="67.945" y1="67.945" x2="74.815" y2="67.945" width="0.254" layer="1"/>
+<wire x1="70.739" y1="67.945" x2="67.945" y2="67.945" width="0.254" layer="1"/>
+<wire x1="77.9" y1="64.86" x2="76.745" y2="64.86" width="0.254" layer="1"/>
+<wire x1="73.025" y1="65.659" x2="70.739" y2="67.945" width="0.254" layer="1"/>
+<wire x1="76.745" y1="64.86" x2="75.946" y2="65.659" width="0.254" layer="1"/>
+<wire x1="75.946" y1="65.659" x2="73.025" y2="65.659" width="0.254" layer="1"/>
 </signal>
 <signal name="LED_B">
@@
 <contactref element="U2" pad="P$12"/>
 <contactref element="C7" pad="1"/>
-<wire x1="74.62" y1="30.74" x2="74.62" y2="36.205" width="0.4064" layer="1"/>
 <contactref element="C13" pad="+"/>
-<wire x1="60.65" y1="30.74" x2="60.65" y2="35.824" width="0.4064" layer="1"/>
-<wire x1="60.65" y1="35.824" x2="60.96" y2="36.134" width="0.4064" layer="1"/>
-<wire x1="74.62" y1="36.205" x2="74.93" y2="36.261" width="0.4064" layer="1"/>
 <wire x1="74.93" y1="36.261" x2="78.735" y2="36.261" width="0.4064" layer="1"/>
 <wire x1="78.735" y1="36.261" x2="78.74" y2="36.256" width="0.4064" layer="1"/>
-<wire x1="21.45" y1="36.69" x2="24.765" y2="36.69" width="0.8128" layer="1"/>
-<wire x1="12.573" y1="25.015" x2="12.573" y2="27.813" width="0.8128" layer="1"/>
-<wire x1="12.573" y1="27.813" x2="21.45" y2="36.69" width="0.8128" layer="1"/>
 <wire x1="24.765" y1="36.69" x2="29.845" y2="36.69" width="0.6096" layer="1"/>
 <wire x1="29.845" y1="36.69" x2="30.48" y2="36.69" width="0.6096" layer="1"/>
 <wire x1="30.48" y1="36.69" x2="57.29" y2="36.69" width="0.6096" layer="1"/>
-<wire x1="57.846" y1="36.134" x2="60.96" y2="36.134" width="0.6096" layer="1"/>
-<wire x1="57.29" y1="36.69" x2="57.846" y2="36.134" width="0.6096" layer="1"/>
-<wire x1="60.96" y1="36.134" x2="60.965" y2="36.129" width="0.6096" layer="1"/>
-<wire x1="60.965" y1="36.129" x2="64.77" y2="36.129" width="0.6096" layer="1"/>
-<wire x1="64.77" y1="36.129" x2="74.798" y2="36.129" width="0.6096" layer="1"/>
-<wire x1="74.798" y1="36.129" x2="74.93" y2="36.261" width="0.6096" layer="1"/>
 <wire x1="29.983" y1="36.828" x2="29.845" y2="36.69" width="0.254" layer="1"/>
 <wire x1="27.2749" y1="44.765" x2="23.749" y2="44.765" width="0.508" layer="1"/>
@@
 <wire x1="30.618" y1="40.005" x2="30.618" y2="36.828" width="0.254" layer="1"/>
 <wire x1="30.618" y1="36.828" x2="30.48" y2="36.69" width="0.254" layer="1"/>
+<wire x1="12.573" y1="25.015" x2="12.573" y2="27.813" width="1.016" layer="1"/>
+<wire x1="12.573" y1="27.813" x2="21.45" y2="36.69" width="1.016" layer="1"/>
+<wire x1="21.45" y1="36.69" x2="24.765" y2="36.69" width="1.016" layer="1"/>
+<wire x1="24.765" y1="36.69" x2="57.29" y2="36.69" width="1.016" layer="1"/>
+<wire x1="57.29" y1="36.69" x2="57.846" y2="36.134" width="1.016" layer="1"/>
+<wire x1="57.846" y1="36.134" x2="60.96" y2="36.134" width="1.016" layer="1"/>
+<wire x1="60.96" y1="36.134" x2="64.765" y2="36.134" width="1.016" layer="1"/>
+<wire x1="64.765" y1="36.134" x2="64.77" y2="36.129" width="1.016" layer="1"/>
+<wire x1="64.77" y1="36.129" x2="74.798" y2="36.129" width="1.016" layer="1"/>
+<wire x1="74.798" y1="36.129" x2="74.93" y2="36.261" width="1.016" layer="1"/>
+<wire x1="60.65" y1="30.74" x2="60.65" y2="32.964" width="0.4064" layer="1"/>
+<wire x1="60.96" y1="33.655" x2="60.96" y2="36.134" width="0.6096" layer="1"/>
+<wire x1="74.93" y1="33.655" x2="74.93" y2="36.261" width="0.6096" layer="1"/>
+<wire x1="74.62" y1="30.74" x2="74.62" y2="32.71" width="0.4064" layer="1"/>
+<wire x1="74.62" y1="32.71" x2="74.93" y2="33.02" width="0.4064" layer="1"/>
+<wire x1="74.93" y1="33.02" x2="74.93" y2="33.655" width="0.4064" layer="1"/>
+<wire x1="60.96" y1="33.274" x2="60.96" y2="33.655" width="0.4064" layer="1"/>
+<wire x1="60.65" y1="32.964" x2="60.96" y2="33.274" width="0.4064" layer="1"/>
 </signal>
 <signal name="DTR">
@@
 <wire x1="8.899" y1="12.065" x2="8.899" y2="10.091" width="0.8128" layer="1"/>
 <wire x1="10.13" y1="8.86" x2="10.13" y2="6.35" width="0.8128" layer="1"/>
-<wire x1="5.715" y1="49.1236" x2="5.715" y2="46.99" width="0.8128" layer="1"/>
-<wire x1="5.715" y1="46.99" x2="6.35" y2="46.355" width="0.8128" layer="1"/>
-<wire x1="6.35" y1="46.355" x2="10.16" y2="46.355" width="0.8128" layer="1"/>
-<wire x1="10.16" y1="46.355" x2="10.795" y2="45.72" width="0.8128" layer="1"/>
-<wire x1="10.795" y1="45.72" x2="10.795" y2="43.815" width="0.8128" layer="1"/>
 <wire x1="6.08" y1="15.56" x2="8.945" y2="15.56" width="0.254" layer="1"/>
 <wire x1="8.945" y1="15.56" x2="9.006" y2="15.621" width="0.254" layer="1"/>
 <wire x1="9.006" y1="15.621" x2="8.899" y2="15.514" width="0.254" layer="1"/>
 <wire x1="8.899" y1="15.514" x2="8.899" y2="12.065" width="0.254" layer="1"/>
-<wire x1="10.795" y1="43.815" x2="10.795" y2="40.64" width="0.8128" layer="1"/>
-<wire x1="10.795" y1="40.64" x2="7.62" y2="37.465" width="0.8128" layer="1"/>
 <wire x1="5.08" y1="12.065" x2="8.899" y2="12.065" width="0.8128" layer="1"/>
-<wire x1="7.62" y1="37.465" x2="7.62" y2="30.48" width="0.8128" layer="1"/>
-<wire x1="7.62" y1="30.48" x2="2.286" y2="25.146" width="0.8128" layer="1"/>
-<wire x1="2.286" y1="25.146" x2="2.286" y2="14.859" width="0.8128" layer="1"/>
-<wire x1="2.286" y1="14.859" x2="5.08" y2="12.065" width="0.8128" layer="1"/>
+<wire x1="5.08" y1="12.065" x2="2.286" y2="14.859" width="0.8128" layer="1"/>
+<wire x1="2.286" y1="14.859" x2="2.286" y2="40.64" width="0.8128" layer="1"/>
+<wire x1="2.286" y1="40.64" x2="2.286" y2="47.371" width="0.8128" layer="1"/>
+<wire x1="4.0386" y1="49.1236" x2="5.715" y2="49.1236" width="0.8128" layer="1"/>
+<wire x1="2.286" y1="47.371" x2="4.0386" y2="49.1236" width="0.8128" layer="1"/>
+<wire x1="10.795" y1="43.815" x2="10.795" y2="42.545" width="0.8128" layer="1"/>
+<wire x1="10.795" y1="42.545" x2="8.89" y2="40.64" width="0.8128" layer="1"/>
+<wire x1="8.89" y1="40.64" x2="2.286" y2="40.64" width="0.8128" layer="1"/>
 </signal>
 <signal name="RESET">
@@
 <contactref element="F1" pad="1"/>
 <contactref element="D2" pad="C"/>
-<wire x1="13.199" y1="12.065" x2="13.199" y2="18.809" width="0.8128" layer="1"/>
-<wire x1="13.199" y1="18.809" x2="12.573" y2="19.435" width="0.8128" layer="1"/>
+<wire x1="12.829" y1="19.179" x2="12.573" y2="19.435" width="0.8128" layer="1"/>
 <wire x1="6.08" y1="17.46" x2="7.935" y2="17.46" width="0.8128" layer="1"/>
 <wire x1="9.91" y1="19.435" x2="12.573" y2="19.435" width="0.8128" layer="1"/>
 <wire x1="7.935" y1="17.46" x2="9.91" y2="19.435" width="0.8128" layer="1"/>
+<wire x1="13.199" y1="12.065" x2="13.199" y2="18.809" width="1.016" layer="1"/>
+<wire x1="13.199" y1="18.809" x2="12.829" y2="19.179" width="1.016" layer="1"/>
 </signal>
 <signal name="N$4">
