File: Devboard_1.1/devboard.sch (EAGLE design)
At the start: 89 parts, among them J1 USB-MICROB-2, J10 MJ-2509N, J11 MJ-2509N, J12 MJ-2509N, J13 MJ-2509N, J14 1x8M, J15 1x8F, J16 1x8F, J17 1x2M, J2 1x2M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

Commit message: Updates to 1.1 board
Parts:
- added C12: 10uF, vibhud:CAPACITOR-1206
- added D3: Blue, vibhud:LED0805-NO_OUTLINE
- added R10: 51R, vibhud:RESISTOR0805
- added R11: 1k, vibhud:RESISTOR0805
- added U5: PCA9634D, vibhud:PCA963420-TSSOP
- RN1, RN2, RN3, RN4, RN5, RN6, RN7, RN8, RN9: device vibhud:4R-NEXBS8V -> vibhud:4R-NEXB38V
Connections:
- new net N$12: D1.A, R10.1
- new net N$13: D3.A, R11.2
- new net N$14: J13.TS, J9.VBUS
- new net N$32: J10.TS, J6.VBUS
- new net N$33: J11.TS, J7.VBUS
- new net N$34: J12.TS, J8.VBUS
- net 3.3V: now also C12.1, R10.2, U5.VDD; no longer D1.A
- net GND: now also C12.2, D3.C, U5.A0, U5.A1, U5.A2, U5.A3, U5.A4, U5.A5, U5.A6, U5.GND, U5.OE
- net GPIO15: now also R11.1
- net MOT_0P: no longer J6.VBUS
- net MOT_1N: now also U2.B_OUT2; no longer U2.B_OUT1
- net MOT_1P: now also U2.B_OUT1; no longer J7.VBUS, U2.B_OUT2
- net MOT_2P: no longer J8.VBUS
- net MOT_3N: now also U3.B_OUT2; no longer U3.B_OUT1
- net MOT_3P: now also U3.B_OUT1; no longer J9.VBUS, U3.B_OUT2
- net PWM0: now also U5.LED0
- net PWM1: now also U5.LED1
- net PWM2: now also U5.LED2
- net PWM3: now also U5.LED3
- net PWM4: now also U5.LED4
- net PWM5: now also U5.LED5
- net PWM6: now also U5.LED6
- net PWM7: now also U5.LED7
- net SCL: now also U5.SCL
- net SDA: now also U5.SDA
Other:
- moved on the sheet: J10, J11, J12, J13
