File: Devboard_1.1/devboard.sch (EAGLE design)
At the start: 94 parts, among them J1 USB-MICROB-2, J10 MJ-2509N, J11 MJ-2509N, J12 MJ-2509N, J13 MJ-2509N, J14 1x8M, J15 1x8F, J16 1x8F, J17 1x2M, J2 1x2M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

Commit message: Updated 1.1 board
Parts:
- removed C12: 10uF, vibhud:CAPACITOR-1206
- removed J17: 1x2M, vibhud:CONN_02LOCK_LONGPADS
- removed U5: PCA9634D, vibhud:PCA963420-TSSOP
- added J19: 1x8M, vibhud:CONN_06LOCK
- C1, C10, C11, C2, C3, C4, C5, C6, C7, C8, C9: device vibhud:CAPACITOR-1206 -> vibhud:CAPACITOR-0805
- RN1, RN2, RN3, RN4, RN5, RN7, RN8, RN9: device vibhud:4R-NEXB38V -> vibhud:4R-NEXB28V
- RN6: device vibhud:4R-NEXB38V -> vibhud:4R-NEXBN8V
Connections:
- removed net N$31: J16.1, J17.2
- net 3.3V: no longer C12.1, U5.VDD
- net CH_PD: now also RN8C.2; no longer RN8B.2
- net GND: now also J19.1; no longer C12.2, U5.A0, U5.A1, U5.A2, U5.A3, U5.A4, U5.A5, U5.A6, U5.GND, U5.OE
- net GPIO0: now also RN8A.2; no longer RN8D.2
- net GPIO14: now also RN8D.2; no longer RN8C.2
- net PWM0: no longer U5.LED0
- net PWM1: no longer U5.LED1
- net PWM2: no longer U5.LED2
- net PWM3: no longer U5.LED3
- net PWM4: no longer U5.LED4
- net PWM5: no longer U5.LED5
- net PWM6: no longer U5.LED6
- net PWM7: no longer U5.LED7
- net RESET: now also RN8B.2; no longer RN8A.2
- net SCL: no longer U5.SCL
- net SDA: no longer U5.SDA
- net TXD0: now also J19.5
- net USB_RXD: now also J19.4
- net V_USB: now also J16.1, J19.3; no longer J17.1
Other:
- moved on the sheet: RN8A, RN8B, RN8C, RN8D

Commit message: Updates to 1.1 board
Parts:
- added U$1: DICKBUTT, vibhud:DICKBUTT
- F1: value 6V/2A -> 16V/2.2A; device vibhud:PPTC_HALF-AMP -> vibhud:PPTC1812
- RN6: device vibhud:4R-NEXBN8V -> vibhud:4R-NEXB28V
- renumbered J19 to FTDI
Connections:
- net 3.3V: now also U1.A5, U1.A6
- net GND: no longer U1.A5, U1.A6

Commit message: 1.1 board finalizations
Parts:
- added U$2: JASX_LOGO_LARGE, vibhud:JASX_LOGO_LARGE
- U$1: value DICKBUTT -> DICKBUTTCOPPER; device vibhud:DICKBUTT -> vibhud:DICKBUTTCOPPER
Changed lines of the file:
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@@
 <grid distance="0.1" unitdist="inch" unit="inch" style="lines" multiple="1" display="no" altdistance="0.01" altunitdist="inch" altunit="inch"/>
 <layers>
-<layer number="1" name="Top" color="4" fill="1" visible="no" active="no"/>
-<layer number="16" name="Bottom" color="1" fill="1" visible="no" active="no"/>
-<layer number="17" name="Pads" color="2" fill="1" visible="no" active="no"/>
-<layer number="18" name="Vias" color="2" fill="1" visible="no" active="no"/>
-<layer number="19" name="Unrouted" color="6" fill="1" visible="no" active="no"/>
-<layer number="20" name="Dimension" color="24" fill="1" visible="no" active="no"/>
-<layer number="21" name="tPlace" color="7" fill="1" visible="no" active="no"/>
-<layer number="22" name="bPlace" color="7" fill="1" visible="no" active="no"/>
-<layer number="23" name="tOrigins" color="15" fill="1" visible="no" active="no"/>
-<layer number="24" name="bOrigins" color="15" fill="1" visible="no" active="no"/>
-<layer number="25" name="tNames" color="7" fill="1" visible="no" active="no"/>
-<layer number="26" name="bNames" color="7" fill="1" visible="no" active="no"/>
-<layer number="27" name="tValues" color="7" fill="1" visible="no" active="no"/>
-<layer number="28" name="bValues" color="7" fill="1" visible="no" active="no"/>
+<layer number="1" name="Top" color="4" fill="1" visible="yes" active="no"/>
+<layer number="16" name="Bottom" color="1" fill="1" visible="yes" active="no"/>
+<layer number="17" name="Pads" color="2" fill="1" visible="yes" active="no"/>
+<layer number="18" name="Vias" color="2" fill="1" visible="yes" active="no"/>
+<layer number="19" name="Unrouted" color="6" fill="1" visible="yes" active="no"/>
+<layer number="20" name="Dimension" color="24" fill="1" visible="yes" active="no"/>
+<layer number="21" name="tPlace" color="7" fill="1" visible="yes" active="no"/>
+<layer number="22" name="bPlace" color="7" fill="1" visible="yes" active="no"/>
+<layer number="23" name="tOrigins" color="15" fill="1" visible="yes" active="no"/>
+<layer number="24" name="bOrigins" color="15" fill="1" visible="yes" active="no"/>
+<layer number="25" name="tNames" color="7" fill="1" visible="yes" active="no"/>
+<layer number="26" name="bNames" color="7" fill="1" visible="yes" active="no"/>
+<layer number="27" name="tValues" color="7" fill="1" visible="yes" active="no"/>
+<layer number="28" name="bValues" color="7" fill="1" visible="yes" active="no"/>
 <layer number="29" name="tStop" color="7" fill="3" visible="no" active="no"/>
 <layer number="30" name="bStop" color="7" fill="6" visible="no" active="no"/>
@@
 <layer number="35" name="tGlue" color="7" fill="4" visible="no" active="no"/>
 <layer number="36" name="bGlue" color="7" fill="5" visible="no" active="no"/>
-<layer number="37" name="tTest" color="7" fill="1" visible="no" active="no"/>
-<layer number="38" name="bTest" color="7" fill="1" visible="no" active="no"/>
+<layer number="37" name="tTest" color="7" fill="1" visible="yes" active="no"/>
+<layer number="38" name="bTest" color="7" fill="1" visible="yes" active="no"/>
 <layer number="39" name="tKeepout" color="4" fill="11" visible="no" active="no"/>
 <layer number="40" name="bKeepout" color="1" fill="11" visible="no" active="no"/>
@@
 <layer number="44" name="Drills" color="7" fill="1" visible="no" active="no"/>
 <layer number="45" name="Holes" color="7" fill="1" visible="no" active="no"/>
-<layer number="46" name="Milling" color="3" fill="1" visible="no" active="no"/>
-<layer number="47" name="Measures" color="7" fill="1" visible="no" active="no"/>
-<layer number="48" name="Document" color="7" fill="1" visible="no" active="no"/>
-<layer number="49" name="Reference" color="7" fill="1" visible="no" active="no"/>
-<layer number="50" name="dxf" color="7" fill="1" visible="no" active="no"/>
-<layer number="51" name="tDocu" color="7" fill="1" visible="no" active="no"/>
-<layer number="52" name="bDocu" color="7" fill="1" visible="no" active="no"/>
-<layer number="53" name="tGND_GNDA" color="7" fill="9" visible="no" active="no"/>
-<layer number="54" name="bGND_GNDA" color="1" fill="9" visible="no" active="no"/>
-<layer number="56" name="wert" color="7" fill="1" visible="no" active="no"/>
-<layer number="57" name="tCAD" color="7" fill="1" visible="no" active="no"/>
-<layer number="59" name="tCarbon" color="7" fill="1" visible="no" active="no"/>
-<layer number="60" name="bCarbon" color="7" fill="1" visible="no" active="no"/>
+<layer number="46" name="Milling" color="3" fill="1" visible="yes" active="no"/>
+<layer number="47" name="Measures" color="7" fill="1" visible="yes" active="no"/>
+<layer number="48" name="Document" color="7" fill="1" visible="yes" active="no"/>
+<layer number="49" name="Reference" color="7" fill="1" visible="yes" active="no"/>
+<layer number="50" name="dxf" color="7" fill="1" visible="yes" active="no"/>
+<layer number="51" name="tDocu" color="7" fill="1" visible="yes" active="no"/>
+<layer number="52" name="bDocu" color="7" fill="1" visible="yes" active="no"/>
+<layer number="53" name="tGND_GNDA" color="7" fill="9" visible="yes" active="no"/>
+<layer number="54" name="bGND_GNDA" color="1" fill="9" visible="yes" active="no"/>
+<layer number="56" name="wert" color="7" fill="1" visible="yes" active="no"/>
+<layer number="57" name="tCAD" color="7" fill="1" visible="yes" active="no"/>
+<layer number="59" name="tCarbon" color="7" fill="1" visible="yes" active="no"/>
+<layer number="60" name="bCarbon" color="7" fill="1" visible="yes" active="no"/>
 <layer number="88" name="SimResults" color="9" fill="1" visible="yes" active="yes"/>
 <layer number="89" name="SimProbes" color="9" fill="1" visible="yes" active="yes"/>
@@
 <part name="SUPPLY8" library="vibhud" library_urn="urn:adsk.eagle:library:2530795" deviceset="V_USB" device=""/>
 <part name="GND10" library="vibhud" library_urn="urn:adsk.eagle:library:2530795" deviceset="GND" device=""/>
-<part name="U$1" library="vibhud" library_urn="urn:adsk.eagle:library:2530795" deviceset="DICKBUTT" device=""/>
+<part name="U$2" library="vibhud" library_urn="urn:adsk.eagle:library:2530795" deviceset="JASX_LOGO" device="_LARGE" value="JASX_LOGO_LARGE"/>
+<part name="U$1" library="vibhud" library_urn="urn:adsk.eagle:library:2530795" deviceset="DICKBUTT" device="COPPER"/>
 </parts>
 <sheets>
@@
 <instance part="GND6" gate="1" x="104.14" y="17.78"/>
 <instance part="R11" gate="G$1" x="88.9" y="22.86"/>
-<instance part="U$1" gate="G$1" x="15.24" y="17.78"/>
+<instance part="U$2" gate="G$1" x="15.24" y="25.4"/>
+<instance part="U$1" gate="G$2" x="-81.28" y="83.82"/>
 </instances>
 <busses>
